Commit message: Feature modifications for mechanical sonar: 	- Rotation of the link 	- Modification of the horizontal FOV 	- Ploting with image compostion

File: xacro/base_car_sonar.xacro (robot description, xacro)
@@ -66,10 +66,9 @@
       </collision>
     </link>
-    <joint name="${namespace}/test_joint" type="revolute">
-      <origin xyz="0 0 3" rpy="0 ${pi/2} ${pi/2}"/>
+    <joint name="${namespace}/test_joint" type="continuous">
+      <origin xyz="0 0 0.5" rpy="0 0 0"/>
+      <axis xyz="0 0 1" />
       <parent link="${namespace}/base_link" />
       <child link="${namespace}/test_link" />
-      <limit upper="0" lower="0" effort="0" velocity="0" />
-      <axis xyz="1 0 0"/>
     </joint>
     <!-- Set up hydrodynamic plugin given as input parameter -->

File: xacro/default_car_sonar.xacro (robot description, xacro)
@@ -6,6 +6,6 @@
   <!-- -->
   <!-- Include the ROV macro file -->
-  <xacro:include filename="$(find foward_looking_gazebo_sonar)/xacro/base_$(arg concept).xacro"/>
-  <xacro:include filename="$(find foward_looking_gazebo_sonar)/xacro/gazebo_$(arg concept).xacro"/>
+  <xacro:include filename="$(find mechanical_scanning_imaging_sonar)/xacro/base_$(arg concept).xacro"/>
+  <xacro:include filename="$(find mechanical_scanning_imaging_sonar)/xacro/gazebo_$(arg concept).xacro"/>
   <!-- -->
   <!-- Create the car_sonar -->

File: xacro/gazebo_car_sonar.xacro (robot description, xacro)
@@ -4,19 +4,29 @@
 <sensor name='MSISonar' type='camera'>
     <plugin name="SonarVisual" filename="libMechanicalScanningImagingSonarGazebo.so" >
+        <update_rate>10</update_rate>
         <topic>car_sonar/MSISonar</topic>
         <debug>1</debug>
+        <axis_rotation>2</axis_rotation>
+        <angle_max>${pi/4}</angle_max>
+        <angle_min>${-pi/4}</angle_min>
+        <axis_rotation>2</axis_rotation>
+        <angular_velocity>${pi/4}</angular_velocity>
         <link_reference>car_sonar/test_link</link_reference>
         <horizontal_fov>${pi/2}</horizontal_fov>
         <vfov>${pi/4}</vfov>
         <bin_count>720</bin_count>
-        <beam_count>720</beam_count>
+        <beam_count>20</beam_count>
         <image>
-            <width>720</width>
+            <width>20</width>
             <height>720</height>
             <format>R32G32B32</format>
         </image>
+        <sonar_output>
+            <width>720</width>
+            <height>720</height>
+        </sonar_output>
         <clip>
             <near>0.1</near>
-            <far>5</far>
+            <far>4</far>
         </clip>
         <noise>

Commit message: Problems correction (DownTilting,ImageComposition): 	- Downtilting is now seeing correctly 	- Image composition

File: xacro/base_car_sonar.xacro (robot description, xacro)
@@ -14,4 +14,5 @@
   <!-- Fluid density -->
   <xacro:property name="rho" value="1028"/>
+  <link name="world"/>
   <!-- Vehicle macro -->
   <xacro:macro name="car_sonar_base" params="namespace *gazebo">
@@ -72,4 +73,9 @@
       <child link="${namespace}/test_link" />
     </joint>
+    <joint name="${namespace}/fixed_joint" type="fixed">
+      <origin xyz="0 0 6" rpy="0 ${0} 0"/>
+      <parent link="world" />
+      <child link="${namespace}/base_link" />
+    </joint>
     <!-- Set up hydrodynamic plugin given as input parameter -->
     <xacro:insert_block name="gazebo"/>

File: xacro/gazebo_car_sonar.xacro (robot description, xacro)
@@ -2,22 +2,59 @@
 <robot xmlns:xacro="http://www.ros.org/wiki/xacro">
 <gazebo reference="car_sonar/test_link">
+<!-- <sensor name='MSISonar' type='camera'>
+    <plugin name="SonarVisual" filename="libMechanicalScanningImagingSonarGazebo.so" >
+        <update_rate>15</update_rate>
+        <local_rotation>${20*pi/180} 0 0</local_rotation>
+        <topic>car_sonar/MSISonar</topic>
+        <debug>0</debug>
+        <axis_rotation>2</axis_rotation>
+        <angle_max>${120*pi/180}</angle_max>
+        <angle_min>${-120*pi/180}</angle_min>
+        <axis_rotation>2</axis_rotation>
+        <angular_velocity>${pi/4}</angular_velocity>
+        <link_reference>car_sonar/test_link</link_reference>
+        <hfov>${3*pi/180}</hfov>
+        <vfov>${35*pi/180}</vfov>
+        <bin_count>1350</bin_count>
+        <beam_count>1</beam_count>
+        <image>
+            <width>10</width>
+            <height>1350</height>
+            <format>R32G32B32</format>
+        </image>
+        <sonar_output>
+            <width>1080</width>
+            <height>1080</height>
+        </sonar_output>
+        <clip>
+            <near>0.3</near>
+            <far>75</far>
+        </clip>
+        <noise>
+            <type>gaussian</type>
+            <mean>0.0</mean>
+            <stddev>0.1</stddev>
+        </noise>
+    </plugin>
+</sensor>   -->
 <sensor name='MSISonar' type='camera'>
     <plugin name="SonarVisual" filename="libMechanicalScanningImagingSonarGazebo.so" >
-        <update_rate>10</update_rate>
+        <update_rate>100</update_rate>
+        <local_rotation>0 ${pi/5} 0</local_rotation>
         <topic>car_sonar/MSISonar</topic>
         <debug>1</debug>
         <axis_rotation>2</axis_rotation>
-        <angle_max>${pi/4}</angle_max>
-        <angle_min>${-pi/4}</angle_min>
+        <angle_max>${120*pi/180}</angle_max>
+        <angle_min>${-120*pi/180}</angle_min>
         <axis_rotation>2</axis_rotation>
-        <angular_velocity>${pi/4}</angular_velocity>
+        <angular_velocity>${0.5*pi/6}</angular_velocity>
         <link_reference>car_sonar/test_link</link_reference>
-        <horizontal_fov>${pi/2}</horizontal_fov>
-        <vfov>${pi/4}</vfov>
-        <bin_count>720</bin_count>
-        <beam_count>20</beam_count>
+        <hfov>${3*pi/180}</hfov>
+        <vfov>${35*pi/180}</vfov>
+        <bin_count>1035</bin_count>
+        <beam_count>1</beam_count>
         <image>
-            <width>20</width>
-            <height>720</height>
+            <width>180</width>
+            <height>1035</height>
             <format>R32G32B32</format>
         </image>
@@ -27,6 +64,6 @@
         </sonar_output>
         <clip>
-            <near>0.1</near>
-            <far>4</far>
+            <near>0.3</near>
+            <far>80</far>
         </clip>
         <noise>

Commit message: Correction of angle rotation and readme file

File: xacro/base_car_sonar.xacro (robot description, xacro)
@@ -4,9 +4,9 @@
   <xacro:property name="concept" value="car_sonar"/>
   <!-- Loading vehicle's specific macros -->
-  <xacro:include filename="$(find  foward_looking_gazebo_sonar)/xacro/snippets_${concept}.xacro"/>
+  <xacro:include filename="$(find  mechanical_scanning_imaging_sonar)/xacro/snippets_${concept}.xacro"/>
   <!--
     Vehicle's parameters (remember to enter the model parameters below)
   -->
-  <xacro:property name="visual_mesh_file" value="file://$(find  foward_looking_gazebo_sonar)/meshes/Body_${concept}.stl"/>
+  <xacro:property name="visual_mesh_file" value="file://$(find  mechanical_scanning_imaging_sonar)/meshes/Body_${concept}.stl"/>
   <!-- Loading the UUV simulator ROS plugin macros -->
   <xacro:property name="mass" value="1000"/>
@@ -74,5 +74,5 @@
     </joint>
     <joint name="${namespace}/fixed_joint" type="fixed">
-      <origin xyz="0 0 6" rpy="0 ${0} 0"/>
+      <origin xyz="3.5 -1 5" rpy="0 ${0*pi/10} 0"/>
       <parent link="world" />
       <child link="${namespace}/base_link" />
@@ -81,7 +81,7 @@
     <xacro:insert_block name="gazebo"/>
     <!-- Include the thruster modules -->
-    <xacro:include filename="$(find foward_looking_gazebo_sonar)/xacro/actuators_car_sonar.xacro"/>
+    <xacro:include filename="$(find mechanical_scanning_imaging_sonar)/xacro/actuators_car_sonar.xacro"/>
     <!-- Include the sensor modules -->
-    <xacro:include filename="$(find foward_looking_gazebo_sonar)/xacro/sensors_car_sonar.xacro"/>
+    <xacro:include filename="$(find mechanical_scanning_imaging_sonar)/xacro/sensors_car_sonar.xacro"/>
   </xacro:macro>
 </robot>

File: xacro/gazebo_car_sonar.xacro (robot description, xacro)
@@ -2,44 +2,8 @@
 <robot xmlns:xacro="http://www.ros.org/wiki/xacro">
 <gazebo reference="car_sonar/test_link">
-<!-- <sensor name='MSISonar' type='camera'>
-    <plugin name="SonarVisual" filename="libMechanicalScanningImagingSonarGazebo.so" >
-        <update_rate>15</update_rate>
-        <local_rotation>${20*pi/180} 0 0</local_rotation>
-        <topic>car_sonar/MSISonar</topic>
-        <debug>0</debug>
-        <axis_rotation>2</axis_rotation>
-        <angle_max>${120*pi/180}</angle_max>
-        <angle_min>${-120*pi/180}</angle_min>
-        <axis_rotation>2</axis_rotation>
-        <angular_velocity>${pi/4}</angular_velocity>
-        <link_reference>car_sonar/test_link</link_reference>
-        <hfov>${3*pi/180}</hfov>
-        <vfov>${35*pi/180}</vfov>
-        <bin_count>1350</bin_count>
-        <beam_count>1</beam_count>
-        <image>
-            <width>10</width>
-            <height>1350</height>
-            <format>R32G32B32</format>
-        </image>
-        <sonar_output>
-            <width>1080</width>
-            <height>1080</height>
-        </sonar_output>
-        <clip>
-            <near>0.3</near>
-            <far>75</far>
-        </clip>
-        <noise>
-            <type>gaussian</type>
-            <mean>0.0</mean>
-            <stddev>0.1</stddev>
-        </noise>
-    </plugin>
-</sensor>   -->
 <sensor name='MSISonar' type='camera'>
     <plugin name="SonarVisual" filename="libMechanicalScanningImagingSonarGazebo.so" >
         <update_rate>100</update_rate>
-        <local_rotation>0 ${pi/5} 0</local_rotation>
+        <local_rotation>0 ${1*pi/10} 0</local_rotation>
         <topic>car_sonar/MSISonar</topic>
         <debug>1</debug>
@@ -52,9 +16,9 @@
         <hfov>${3*pi/180}</hfov>
         <vfov>${35*pi/180}</vfov>
-        <bin_count>1035</bin_count>
+        <bin_count>720</bin_count>
         <beam_count>1</beam_count>
         <image>
             <width>180</width>
-            <height>1035</height>
+            <height>720</height>
             <format>R32G32B32</format>
         </image>
@@ -64,6 +28,6 @@
         </sonar_output>
         <clip>
-            <near>0.3</near>
-            <far>80</far>
+            <near>3</near>
+            <far>10</far>
         </clip>
         <noise>

Commit message: Correction of tests and set package name to mechanical_scanning_imaging_sonar_gazebo

File: xacro/base_car_sonar.xacro (robot description, xacro)
@@ -4,9 +4,9 @@
   <xacro:property name="concept" value="car_sonar"/>
   <!-- Loading vehicle's specific macros -->
-  <xacro:include filename="$(find  mechanical_scanning_imaging_sonar)/xacro/snippets_${concept}.xacro"/>
+  <xacro:include filename="$(find  mechanical_scanning_imaging_sonar_gazebo)/xacro/snippets_${concept}.xacro"/>
   <!--
     Vehicle's parameters (remember to enter the model parameters below)
   -->
-  <xacro:property name="visual_mesh_file" value="file://$(find  mechanical_scanning_imaging_sonar)/meshes/Body_${concept}.stl"/>
+  <xacro:property name="visual_mesh_file" value="file://$(find  mechanical_scanning_imaging_sonar_gazebo)/meshes/Body_${concept}.stl"/>
   <!-- Loading the UUV simulator ROS plugin macros -->
   <xacro:property name="mass" value="1000"/>
@@ -81,7 +81,7 @@
     <xacro:insert_block name="gazebo"/>
     <!-- Include the thruster modules -->
-    <xacro:include filename="$(find mechanical_scanning_imaging_sonar)/xacro/actuators_car_sonar.xacro"/>
+    <xacro:include filename="$(find mechanical_scanning_imaging_sonar_gazebo)/xacro/actuators_car_sonar.xacro"/>
     <!-- Include the sensor modules -->
-    <xacro:include filename="$(find mechanical_scanning_imaging_sonar)/xacro/sensors_car_sonar.xacro"/>
+    <xacro:include filename="$(find mechanical_scanning_imaging_sonar_gazebo)/xacro/sensors_car_sonar.xacro"/>
   </xacro:macro>
 </robot>

File: xacro/default_car_sonar.xacro (robot description, xacro)
@@ -6,6 +6,6 @@
   <!-- -->
   <!-- Include the ROV macro file -->
-  <xacro:include filename="$(find mechanical_scanning_imaging_sonar)/xacro/base_$(arg concept).xacro"/>
-  <xacro:include filename="$(find mechanical_scanning_imaging_sonar)/xacro/gazebo_$(arg concept).xacro"/>
+  <xacro:include filename="$(find mechanical_scanning_imaging_sonar_gazebo)/xacro/base_$(arg concept).xacro"/>
+  <xacro:include filename="$(find mechanical_scanning_imaging_sonar_gazebo)/xacro/gazebo_$(arg concept).xacro"/>
   <!-- -->
   <!-- Create the car_sonar -->
